File: spectrum.sch (EAGLE design)
At the start: 83 parts, among them IC1 MSGEQ7DIL, IC2 LM358, U1 ATMEGA328P_PDIP

Commit message: moved dip switch & trimmer sets noise
Parts:
- removed RV1: 100k, SparkFun-Electromechanical:POT
- added R10: 10k, SparkFun-Passives:RESISTOR0402-RES
- added R15: 100k, SparkFun-Passives:POTENTIOMETER
- added R17: 1k, SparkFun-Passives:POTENTIOMETER
Connections:
- new net N$32: R10.1, R17.2
- new net NOISE_LVL: R17.P$1, U1.PC1(ADC1)
- net GND: now also R17.1
- net N$29: now also R15.2; no longer RV1.A
- net N$34: now also R15.1; no longer RV1.E
- net RANGE_HI: now also U$1.P$3, U1.PB7(XTAL2/TOSC2); no longer U$1.P$4, U1.PC2(ADC2)
- net RANGE_LO: now also U$1.P$4, U1.PB6(XTAL1/TOSC1); no longer U$1.P$3, U1.PC1(ADC1)
- net VCC: now also R10.2
Other:
- note added: "8Mhz internal RC clock"
- moved on the sheet: C1, R1, U$1
Changed lines of the file:
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@@
 <part name="GND8" library="SparkFun-Aesthetics" deviceset="GND" device=""/>
 <part name="C7" library="SparkFun-Capacitors" deviceset="CAP" device="0402-CAP" value="0.01uF"/>
-<part name="RV1" library="SparkFun-Electromechanical" deviceset="POT" device="" value="100k"/>
 <part name="U$1" library="SparkFun-Electromechanical" deviceset="2-POS-DIP" device=""/>
+<part name="R10" library="SparkFun-Passives" deviceset="RESISTOR" device="0402-RES" value="10k"/>
+<part name="R15" library="SparkFun-Passives" deviceset="POTENTIOMETER" device="" value="100k"/>
+<part name="R17" library="SparkFun-Passives" deviceset="POTENTIOMETER" device="" value="1k"/>
+<part name="SUPPLY6" library="SparkFun-Aesthetics" deviceset="VCC" device="" value="5V"/>
 <part name="GND9" library="SparkFun-Aesthetics" deviceset="GND" device=""/>
 </parts>
@@
 <sheet>
 <plain>
-<text x="83.82" y="175.26" size="1.778" layer="91">Audio Taper</text>
+<text x="86.36" y="170.18" size="1.778" layer="91">Audio Taper</text>
 <text x="160.02" y="154.94" size="1.778" layer="91">1</text>
 <text x="160.02" y="152.4" size="1.778" layer="91">5</text>
@@
 <text x="53.34" y="50.8" size="1.778" layer="91">d13</text>
 <text x="2.54" y="93.98" size="1.778" layer="91">nc</text>
-<text x="2.54" y="83.82" size="1.778" layer="91">nc</text>
-<text x="2.54" y="78.74" size="1.778" layer="91">nc</text>
 <text x="101.6" y="88.9" size="1.778" layer="91">COL 0</text>
 <text x="119.38" y="86.36" size="1.778" layer="91">COL 1</text>
@@
 <text x="53.34" y="109.22" size="1.778" layer="91">d14</text>
 <text x="53.34" y="96.52" size="1.778" layer="91">A5</text>
+<text x="10.16" y="43.18" size="1.778" layer="91">8Mhz internal RC clock</text>
 </plain>
 <instances>
 <instance part="U1" gate="G$1" x="27.94" y="83.82"/>
-<instance part="SUPPLY1" gate="G$1" x="-7.62" y="121.92"/>
-<instance part="R1" gate="G$1" x="-2.54" y="109.22"/>
-<instance part="C1" gate="G$1" x="-7.62" y="83.82"/>
+<instance part="SUPPLY1" gate="G$1" x="-22.86" y="121.92"/>
+<instance part="R1" gate="G$1" x="-17.78" y="109.22"/>
+<instance part="C1" gate="G$1" x="-22.86" y="93.98"/>
 <instance part="D1" gate="G$1" x="106.68" y="53.34" rot="R270"/>
 <instance part="D2" gate="G$1" x="106.68" y="43.18" rot="R270"/>
@@
 <instance part="D23" gate="G$1" x="142.24" y="-17.78" rot="R270"/>
 <instance part="D24" gate="G$1" x="142.24" y="-27.94" rot="R270"/>
-<instance part="GND1" gate="1" x="-7.62" y="40.64"/>
+<instance part="GND1" gate="1" x="-22.86" y="40.64"/>
 <instance part="R3" gate="G$1" x="93.98" y="38.1"/>
 <instance part="R4" gate="G$1" x="93.98" y="27.94"/>
@@
 <instance part="GND8" gate="1" x="218.44" y="127"/>
 <instance part="C7" gate="G$1" x="129.54" y="152.4" rot="R90"/>
-<instance part="RV1" gate="G$1" x="83.82" y="167.64" rot="R90"/>
-<instance part="U$1" gate="G$1" x="99.06" y="104.14" rot="R90"/>
-<instance part="GND9" gate="1" x="116.84" y="99.06"/>
+<instance part="U$1" gate="G$1" x="-10.16" y="83.82" rot="R270"/>
+<instance part="R10" gate="G$1" x="96.52" y="119.38" rot="R90"/>
+<instance part="R15" gate="G$1" x="83.82" y="167.64"/>
+<instance part="R17" gate="G$1" x="96.52" y="106.68" rot="R90"/>
+<instance part="SUPPLY6" gate="G$1" x="96.52" y="127"/>
+<instance part="GND9" gate="1" x="96.52" y="96.52"/>
 </instances>
 <busses>
@@
 <pinref part="SUPPLY1" gate="G$1" pin="VCC"/>
 <pinref part="R1" gate="G$1" pin="1"/>
-<wire x1="-7.62" y1="121.92" x2="-7.62" y2="109.22" width="0.1524" layer="91"/>
+<wire x1="-22.86" y1="121.92" x2="-22.86" y2="109.22" width="0.1524" layer="91"/>
 <pinref part="U1" gate="G$1" pin="VCC"/>
 <pinref part="U1" gate="G$1" pin="AVCC"/>
 <wire x1="5.08" y1="101.6" x2="5.08" y2="104.14" width="0.1524" layer="91"/>
-<wire x1="5.08" y1="104.14" x2="-7.62" y2="104.14" width="0.1524" layer="91"/>
+<wire x1="5.08" y1="104.14" x2="-22.86" y2="104.14" width="0.1524" layer="91"/>
 <junction x="5.08" y="104.14"/>
-<wire x1="-7.62" y1="104.14" x2="-7.62" y2="109.22" width="0.1524" layer="91"/>
-<junction x="-7.62" y="109.22"/>
+<wire x1="-22.86" y1="104.14" x2="-22.86" y2="109.22" width="0.1524" layer="91"/>
+<junction x="-22.86" y="109.22"/>
 <pinref part="C1" gate="G$1" pin="1"/>
-<wire x1="-7.62" y1="88.9" x2="-7.62" y2="104.14" width="0.1524" layer="91"/>
-<junction x="-7.62" y="104.14"/>
+<wire x1="-22.86" y1="99.06" x2="-22.86" y2="104.14" width="0.1524" layer="91"/>
+<junction x="-22.86" y="104.14"/>
 </segment>
 <segment>
@@
 <wire x1="218.44" y1="190.5" x2="218.44" y2="182.88" width="0.1524" layer="91"/>
 </segment>
+<segment>
+<pinref part="SUPPLY6" gate="G$1" pin="VCC"/>
+<pinref part="R10" gate="G$1" pin="2"/>
+<wire x1="96.52" y1="127" x2="96.52" y2="124.46" width="0.1524" layer="91"/>
+</segment>
 </net>
 <net name="GND" class="0">
@@
 <pinref part="U1" gate="G$1" pin="GND@1"/>
 <wire x1="5.08" y1="53.34" x2="5.08" y2="55.88" width="0.1524" layer="91"/>
-<wire x1="5.08" y1="55.88" x2="-7.62" y2="55.88" width="0.1524" layer="91"/>
+<wire x1="5.08" y1="55.88" x2="-17.78" y2="55.88" width="0.1524" layer="91"/>
 <junction x="5.08" y="55.88"/>
 <pinref part="C1" gate="G$1" pin="2"/>
-<wire x1="-7.62" y1="55.88" x2="-7.62" y2="81.28" width="0.1524" layer="91"/>
+<wire x1="-17.78" y1="55.88" x2="-22.86" y2="55.88" width="0.1524" layer="91"/>
+<wire x1="-22.86" y1="55.88" x2="-22.86" y2="91.44" width="0.1524" layer="91"/>
 <pinref part="GND1" gate="1" pin="GND"/>
-<wire x1="-7.62" y1="55.88" x2="-7.62" y2="43.18" width="0.1524" layer="91"/>
-<junction x="-7.62" y="55.88"/>
+<wire x1="-22.86" y1="55.88" x2="-22.86" y2="43.18" width="0.1524" layer="91"/>
+<junction x="-22.86" y="55.88"/>
+<pinref part="U$1" gate="G$1" pin="P$1"/>
+<pinref part="U$1" gate="G$1" pin="P$2"/>
+<wire x1="-17.78" y1="81.28" x2="-17.78" y2="83.82" width="0.1524" layer="91"/>
+<wire x1="-17.78" y1="81.28" x2="-17.78" y2="55.88" width="0.1524" layer="91"/>
+<junction x="-17.78" y="81.28"/>
+<junction x="-17.78" y="55.88"/>
 </segment>
 <segment>
@@
 </segment>
 <segment>
-<pinref part="U$1" gate="G$1" pin="P$2"/>
-<pinref part="U$1" gate="G$1" pin="P$1"/>
-<wire x1="106.68" y1="106.68" x2="106.68" y2="104.14" width="0.1524" layer="91"/>
 <pinref part="GND9" gate="1" pin="GND"/>
-<wire x1="106.68" y1="104.14" x2="116.84" y2="104.14" width="0.1524" layer="91"/>
-<wire x1="116.84" y1="104.14" x2="116.84" y2="101.6" width="0.1524" layer="91"/>
-<junction x="106.68" y="104.14"/>
+<pinref part="R17" gate="G$1" pin="1"/>
+<wire x1="96.52" y1="99.06" x2="96.52" y2="101.6" width="0.1524" layer="91"/>
 </segment>
 </net>
@@
 <pinref part="U1" gate="G$1" pin="PC6(/RESET)"/>
 <pinref part="R1" gate="G$1" pin="2"/>
-<wire x1="5.08" y1="109.22" x2="2.54" y2="109.22" width="0.1524" layer="91"/>
+<wire x1="5.08" y1="109.22" x2="-12.7" y2="109.22" width="0.1524" layer="91"/>
 </segment>
 </net>
@@
 <wire x1="93.98" y1="167.64" x2="93.98" y2="154.94" width="0.1524" layer="91"/>
 <junction x="93.98" y="154.94"/>
-<pinref part="RV1" gate="G$1" pin="A"/>
-<wire x1="93.98" y1="167.64" x2="91.44" y2="167.64" width="0.1524" layer="91"/>
+<pinref part="R15" gate="G$1" pin="2"/>
+<wire x1="88.9" y1="167.64" x2="93.98" y2="167.64" width="0.1524" layer="91"/>
 </segment>
 </net>
@@
 <wire x1="63.5" y1="167.64" x2="63.5" y2="157.48" width="0.1524" layer="91"/>
 <junction x="63.5" y="157.48"/>
-<pinref part="RV1" gate="G$1" pin="E"/>
-<wire x1="76.2" y1="167.64" x2="63.5" y2="167.64" width="0.1524" layer="91"/>
+<pinref part="R15" gate="G$1" pin="1"/>
+<wire x1="63.5" y1="167.64" x2="78.74" y2="167.64" width="0.1524" layer="91"/>
 </segment>
 </net>
@@
 <net name="RANGE_LO" class="0">
 <segment>
+<pinref part="U1" gate="G$1" pin="PB6(XTAL1/TOSC1)"/>
+<pinref part="U$1" gate="G$1" pin="P$4"/>
+<wire x1="5.08" y1="83.82" x2="-2.54" y2="83.82" width="0.1524" layer="91"/>
+<label x="0" y="86.36" size="1.778" layer="95"/>
+</segment>
+</net>
+<net name="RANGE_HI" class="0">
+<segment>
+<pinref part="U1" gate="G$1" pin="PB7(XTAL2/TOSC2)"/>
+<pinref part="U$1" gate="G$1" pin="P$3"/>
+<wire x1="5.08" y1="78.74" x2="-2.54" y2="78.74" width="0.1524" layer="91"/>
+<wire x1="-2.54" y1="78.74" x2="-2.54" y2="81.28" width="0.1524" layer="91"/>
+<label x="0" y="73.66" size="1.778" layer="95"/>
+</segment>
+</net>
+<net name="N$32" class="0">
+<segment>
+<pinref part="R17" gate="G$1" pin="2"/>
+<pinref part="R10" gate="G$1" pin="1"/>
+<wire x1="96.52" y1="114.3" x2="96.52" y2="111.76" width="0.1524" layer="91"/>
+</segment>
+</net>
+<net name="NOISE_LVL" class="0">
+<segment>
+<pinref part="R17" gate="G$1" pin="P$1"/>
 <pinref part="U1" gate="G$1" pin="PC1(ADC1)"/>
+<wire x1="91.44" y1="106.68" x2="53.34" y2="106.68" width="0.1524" layer="91"/>
 <label x="58.42" y="106.68" size="1.778" layer="95"/>
-<pinref part="U$1" gate="G$1" pin="P$3"/>
-<wire x1="91.44" y1="106.68" x2="53.34" y2="106.68" width="0.1524" layer="91"/>
-</segment>
-</net>
-<net name="RANGE_HI" class="0">
-<segment>
-<pinref part="U1" gate="G$1" pin="PC2(ADC2)"/>
-<label x="58.42" y="104.14" size="1.778" layer="95"/>
-<pinref part="U$1" gate="G$1" pin="P$4"/>
-<wire x1="91.44" y1="104.14" x2="53.34" y2="104.14" width="0.1524" layer="91"/>
-</segment>
-</net>
+</segment>
+</net>

Commit message: first prototype
Parts:
- added C8: 0.33uF, SparkFun-Capacitors:CAP0402-CAP
- added C9: 0.01uF, SparkFun-Capacitors:CAP0402-CAP
- added D57: 1n4001, diode:1N4004
- added IC3: (no value), v-reg:78LXX
- C4: value 0.01uF -> 0.68uF
- C7: value 0.01uF -> 0.1uF
Connections:
- net GND: now also C8.2, C9.2, IC3.GND, R11.1
- net N$25: now also C4.1; no longer R11.1
- net N$26: now also C8.1, IC3.IN; no longer C4.1, R11.2
- net N$29: now also R15.P$1; no longer R15.2
- net VCC: now also C9.1, IC3.OUT
Other:
- moved on the sheet: C4, R11
Changed lines of the file:
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@@
 <part name="IC1" library="SparkFun-AnalogIC" deviceset="MSGEQ7" device="DIL"/>
 <part name="JP1" library="SparkFun-Connectors" deviceset="AUDIO-JACK" device="1:1"/>
-<part name="R11" library="SparkFun-Passives" deviceset="RESISTOR" device="0402-RES" value="10k"/>
 <part name="GND2" library="SparkFun-Aesthetics" deviceset="GND" device=""/>
 <part name="GND3" library="SparkFun-Aesthetics" deviceset="GND" device=""/>
@@
 <part name="C3" library="SparkFun-Capacitors" deviceset="CAP" device="0402-CAP" value="0.1uF"/>
 <part name="GND6" library="SparkFun-Aesthetics" deviceset="GND" device=""/>
-<part name="C4" library="SparkFun-Capacitors" deviceset="CAP" device="0402-CAP" value="0.01uF"/>
+<part name="C4" library="SparkFun-Capacitors" deviceset="CAP" device="0402-CAP" value="0.68uF"/>
 <part name="R12" library="SparkFun-Passives" deviceset="RESISTOR" device="0402-RES" value="22k"/>
 <part name="R13" library="SparkFun-Passives" deviceset="RESISTOR" device="0402-RES" value="12k"/>
@@
 <part name="SUPPLY5" library="SparkFun-Aesthetics" deviceset="VCC" device="" value="5V"/>
 <part name="GND8" library="SparkFun-Aesthetics" deviceset="GND" device=""/>
-<part name="C7" library="SparkFun-Capacitors" deviceset="CAP" device="0402-CAP" value="0.01uF"/>
+<part name="C7" library="SparkFun-Capacitors" deviceset="CAP" device="0402-CAP" value="0.1uF"/>
 <part name="U$1" library="SparkFun-Electromechanical" deviceset="2-POS-DIP" device=""/>
 <part name="R10" library="SparkFun-Passives" deviceset="RESISTOR" device="0402-RES" value="10k"/>
@@
 <part name="SUPPLY6" library="SparkFun-Aesthetics" deviceset="VCC" device="" value="5V"/>
 <part name="GND9" library="SparkFun-Aesthetics" deviceset="GND" device=""/>
+<part name="R11" library="SparkFun-Passives" deviceset="RESISTOR" device="0402-RES" value="10k"/>
+<part name="IC3" library="v-reg" deviceset="78LXX" device=""/>
+<part name="GND10" library="SparkFun-Aesthetics" deviceset="GND" device=""/>
+<part name="SUPPLY7" library="SparkFun-Aesthetics" deviceset="VCC" device="" value="5V"/>
+<part name="D57" library="diode" deviceset="1N4004" device="" value="1n4001"/>
+<part name="C8" library="SparkFun-Capacitors" deviceset="CAP" device="0402-CAP" value="0.33uF"/>
+<part name="C9" library="SparkFun-Capacitors" deviceset="CAP" device="0402-CAP" value="0.01uF"/>
 </parts>
 <sheets>
 <sheet>
 <plain>
-<text x="86.36" y="170.18" size="1.778" layer="91">Audio Taper</text>
+<text x="83.82" y="175.26" size="1.778" layer="91">Audio Taper</text>
 <text x="160.02" y="154.94" size="1.778" layer="91">1</text>
 <text x="160.02" y="152.4" size="1.778" layer="91">5</text>
@@
 <instance part="IC1" gate="G$1" x="175.26" y="149.86"/>
 <instance part="JP1" gate="G$1" x="-5.08" y="160.02"/>
-<instance part="R11" gate="G$1" x="15.24" y="157.48"/>
 <instance part="GND2" gate="1" x="5.08" y="129.54"/>
 <instance part="GND3" gate="1" x="190.5" y="127"/>
@@
 <instance part="C3" gate="G$1" x="63.5" y="182.88"/>
 <instance part="GND6" gate="1" x="71.12" y="129.54"/>
-<instance part="C4" gate="G$1" x="30.48" y="157.48" rot="R90"/>
+<instance part="C4" gate="G$1" x="25.4" y="157.48" rot="R90"/>
 <instance part="R12" gate="G$1" x="38.1" y="177.8" rot="R90"/>
 <instance part="R13" gate="G$1" x="38.1" y="147.32" rot="R90"/>
@@
 <instance part="SUPPLY6" gate="G$1" x="96.52" y="127"/>
 <instance part="GND9" gate="1" x="96.52" y="96.52"/>
+<instance part="R11" gate="G$1" x="10.16" y="147.32" rot="R90"/>
+<instance part="IC3" gate="1" x="10.16" y="5.08"/>
+<instance part="GND10" gate="1" x="10.16" y="-17.78"/>
+<instance part="SUPPLY7" gate="G$1" x="35.56" y="5.08"/>
+<instance part="D57" gate="1" x="-12.7" y="5.08"/>
+<instance part="C8" gate="G$1" x="-2.54" y="-5.08"/>
+<instance part="C9" gate="G$1" x="22.86" y="-5.08"/>
 </instances>
 <busses>
@@
 <wire x1="96.52" y1="127" x2="96.52" y2="124.46" width="0.1524" layer="91"/>
 </segment>
+<segment>
+<pinref part="IC3" gate="1" pin="OUT"/>
+<wire x1="17.78" y1="5.08" x2="22.86" y2="5.08" width="0.1524" layer="91"/>
+<pinref part="SUPPLY7" gate="G$1" pin="VCC"/>
+<pinref part="C9" gate="G$1" pin="1"/>
+<wire x1="22.86" y1="5.08" x2="35.56" y2="5.08" width="0.1524" layer="91"/>
+<wire x1="22.86" y1="0" x2="22.86" y2="5.08" width="0.1524" layer="91"/>
+<junction x="22.86" y="5.08"/>
+</segment>
 </net>
 <net name="GND" class="0">
@@
 <pinref part="JP1" gate="G$1" pin="SLEEVE"/>
 <wire x1="0" y1="162.56" x2="5.08" y2="162.56" width="0.1524" layer="91"/>
-<wire x1="5.08" y1="162.56" x2="5.08" y2="132.08" width="0.1524" layer="91"/>
+<wire x1="5.08" y1="162.56" x2="5.08" y2="134.62" width="0.1524" layer="91"/>
 <pinref part="GND2" gate="1" pin="GND"/>
+<pinref part="R11" gate="G$1" pin="1"/>
+<wire x1="5.08" y1="134.62" x2="5.08" y2="132.08" width="0.1524" layer="91"/>
+<wire x1="10.16" y1="142.24" x2="10.16" y2="134.62" width="0.1524" layer="91"/>
+<wire x1="10.16" y1="134.62" x2="5.08" y2="134.62" width="0.1524" layer="91"/>
+<junction x="5.08" y="134.62"/>
 </segment>
 <segment>
@@
 <pinref part="R17" gate="G$1" pin="1"/>
 <wire x1="96.52" y1="99.06" x2="96.52" y2="101.6" width="0.1524" layer="91"/>
+</segment>
+<segment>
+<pinref part="IC3" gate="1" pin="GND"/>
+<wire x1="10.16" y1="-2.54" x2="10.16" y2="-12.7" width="0.1524" layer="91"/>
+<pinref part="GND10" gate="1" pin="GND"/>
+<pinref part="C8" gate="G$1" pin="2"/>
+<wire x1="10.16" y1="-12.7" x2="10.16" y2="-15.24" width="0.1524" layer="91"/>
+<wire x1="-2.54" y1="-7.62" x2="-2.54" y2="-12.7" width="0.1524" layer="91"/>
+<wire x1="-2.54" y1="-12.7" x2="10.16" y2="-12.7" width="0.1524" layer="91"/>
+<junction x="10.16" y="-12.7"/>
+<pinref part="C9" gate="G$1" pin="2"/>
+<wire x1="22.86" y1="-7.62" x2="22.86" y2="-12.7" width="0.1524" layer="91"/>
+<wire x1="22.86" y1="-12.7" x2="10.16" y2="-12.7" width="0.1524" layer="91"/>
 </segment>
 </net>
@@
 </segment>
 </net>
-<net name="N$26" class="0">
-<segment>
-<wire x1="20.32" y1="157.48" x2="25.4" y2="157.48" width="0.1524" layer="91"/>
-<pinref part="C4" gate="G$1" pin="1"/>
-<pinref part="R11" gate="G$1" pin="2"/>
-</segment>
-</net>
 <net name="N$28" class="0">
 <segment>
@@
 <pinref part="IC2" gate="G1" pin="OUT"/>
 <wire x1="101.6" y1="154.94" x2="93.98" y2="154.94" width="0.1524" layer="91"/>
+<pinref part="R15" gate="G$1" pin="P$1"/>
 <wire x1="93.98" y1="154.94" x2="81.28" y2="154.94" width="0.1524" layer="91"/>
-<wire x1="93.98" y1="167.64" x2="93.98" y2="154.94" width="0.1524" layer="91"/>
+<wire x1="83.82" y1="172.72" x2="93.98" y2="172.72" width="0.1524" layer="91"/>
+<wire x1="93.98" y1="172.72" x2="93.98" y2="154.94" width="0.1524" layer="91"/>
 <junction x="93.98" y="154.94"/>
-<pinref part="R15" gate="G$1" pin="2"/>
-<wire x1="88.9" y1="167.64" x2="93.98" y2="167.64" width="0.1524" layer="91"/>
 </segment>
 </net>
@@
 <pinref part="R14" gate="G$1" pin="1"/>
 <pinref part="C4" gate="G$1" pin="2"/>
-<wire x1="33.02" y1="157.48" x2="50.8" y2="157.48" width="0.1524" layer="91"/>
+<wire x1="27.94" y1="157.48" x2="50.8" y2="157.48" width="0.1524" layer="91"/>
 </segment>
 </net>
@@
 <net name="N$25" class="0">
 <segment>
-<pinref part="R11" gate="G$1" pin="1"/>
 <pinref part="JP1" gate="G$1" pin="LEFT"/>
 <wire x1="10.16" y1="157.48" x2="0" y2="157.48" width="0.1524" layer="91"/>
+<wire x1="10.16" y1="149.86" x2="10.16" y2="157.48" width="0.1524" layer="91"/>
+<pinref part="C4" gate="G$1" pin="1"/>
+<wire x1="20.32" y1="157.48" x2="10.16" y2="157.48" width="0.1524" layer="91"/>
+<junction x="10.16" y="157.48"/>
 </segment>
 </net>
@@
 </segment>
 </net>
+<net name="9V" class="0">
+<segment>
+<wire x1="-20.32" y1="5.08" x2="-20.32" y2="12.7" width="0.1524" layer="91"/>
+<label x="-20.32" y="12.7" size="1.778" layer="95"/>
+<wire x1="-17.78" y1="5.08" x2="-20.32" y2="5.08" width="0.1524" layer="91"/>
+</segment>
+</net>
+<net name="N$26" class="0">
+<segment>
+<pinref part="IC3" gate="1" pin="IN"/>
+<wire x1="2.54" y1="5.08" x2="-2.54" y2="5.08" width="0.1524" layer="91"/>
+<pinref part="C8" gate="G$1" pin="1"/>
+<wire x1="-2.54" y1="5.08" x2="-7.62" y2="5.08" width="0.1524" layer="91"/>
+<wire x1="-2.54" y1="0" x2="-2.54" y2="5.08" width="0.1524" layer="91"/>
+<junction x="-2.54" y="5.08"/>
+</segment>
+</net>
